File: hardware/station_pcb/_autosave-station_pcb.kicad_sch (KiCad schematic)
At the start: 13 parts, among them J1 Bus_I2C_Commun, J2 Programmateur_ISP, J3 MPU-6050, J4 Conn_Alimentation, U2 ATmega328P-P, Y1 Crystal

Commit message: Documentation Updated
Parts:
- removed J1: Bus_I2C_Commun, Connector_PinHeader_2.54mm:PinHeader_1x04_P2.54mm_Vertical, symbol Connector:Conn_01x04_Pin
- removed J2: Programmateur_ISP, Connector_PinHeader_2.54mm:PinHeader_1x06_P2.54mm_Vertical, symbol Connector:Conn_01x06_Pin
- removed J3: MPU-6050, Connector_PinHeader_2.54mm:PinHeader_1x08_P2.54mm_Vertical, symbol Connector:Conn_01x08_Socket
- removed J4: Conn_Alimentation, Connector_PinHeader_2.54mm:PinHeader_1x02_P2.54mm_Vertical, symbol Connector:Conn_01x02_Pin
- removed U2: ATmega328P-P, Package_DIP:DIP-28_W7.62mm, symbol MCU_Microchip_ATmega:ATmega328P-P
- added J1: Conn_Alimentation, Connector_PinHeader_2.54mm:PinHeader_1x02_P2.54mm_Vertical, symbol Connector:Conn_01x02_Pin
- added J2: Bus_I2C_Commun, Connector_PinHeader_2.54mm:PinHeader_1x04_P2.54mm_Vertical, symbol Connector:Conn_01x04_Pin
- added J3: LCD_I2C, Connector_PinHeader_2.54mm:PinHeader_1x04_P2.54mm_Vertical, symbol Connector:Conn_01x04_Socket
- added J4: Programmateur_ISP, Connector_PinHeader_2.54mm:PinHeader_1x06_P2.54mm_Vertical, symbol Connector:Conn_01x06_Pin
- added U1: ATmega328P-P, Package_DIP:DIP-28_W7.62mm, symbol MCU_Microchip_ATmega:ATmega328P-P
- C1, C2: value 100n -> 22p; footprint Capacitor_THT:CP_Radial_D6.3mm_P2.50mm -> Capacitor_THT:CP_Radial_D5.0mm_P2.50mm
- C3, C4: value 22p -> 100n; footprint Capacitor_THT:CP_Radial_D5.0mm_P2.50mm -> Capacitor_THT:CP_Radial_D6.3mm_P2.50mm
- R2, R3: value 4.7k -> 4k7
Connections:
- net 5V: now also C4.1, R2.1, J1.1 (Pin_1), J2.3 (Pin_3), J3.2 (Pin_2), J4.2 (Pin_2), U1.7 (VCC); no longer C1.2, R2.2
- net GND: now also J1.2 (Pin_2), J2.4 (Pin_4), J3.1 (Pin_1), J4.6 (Pin_6), U1.22 (GND), U1.8 (GND)
- net at R1.2: now also J4.5 (Pin_5), U1.1 (~{RESET}/PC6)
- net at R3.1: now also J2.2 (Pin_2), J3.4 (Pin_4), U1.28 (PC5)
- net at Y1.1: now also C2.2, U1.10 (XTAL2/PB7); no longer C4.1
- net at C3.1: now also U1.20 (AVCC); no longer Y1.2
- new net: J2.1 (Pin_1), J3.3 (Pin_3), R2.2, U1.27 (PC4)
- new net: J4.1 (Pin_1), U1.18 (PB4)
- new net: J4.3 (Pin_3), U1.19 (PB5)
- new net: J4.4 (Pin_4), U1.17 (PB3)
- new net: C1.2, U1.9 (XTAL1/PB6), Y1.2
- no-connect marks 3 -> 0
Other:
- title: BlackBox -> (none)
- moved on the sheet: Y1
